File: hardware/cm.kicad_sch (KiCad schematic)
At the start: 0 parts

Commit message: Rename project to Granit
Other:
- company: https://github.com/laenzlinger/offsite-backup -> https://github.com/laenzlinger/granit
- title: Offsite Backup Device - CM4/CM5 + Ethernet -> Granit — CM4/CM5 + Ethernet
Changed lines of the file:
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@@
 	(paper "A4")
 	(title_block
-		(title "Offsite Backup Device - CM4/CM5 + Ethernet")
+		(title "Granit — CM4/CM5 + Ethernet")
 		(date "2026-04-07")
 		(rev "0.1")
-		(company "https://github.com/laenzlinger/offsite-backup")
+		(company "https://github.com/laenzlinger/granit")
 		(comment 1 "License: CERN Open Hardware Licence Version 2 - Permissive")
 		(comment 2 "Git commit hash: ${GIT_HASH}")
