File: hardware/cm-conn2.kicad_sch (KiCad schematic)
At the start: 0 parts

Commit message: Split CM4 into separate connector sheets, add peripherals sheet
Sheet structure:
- psu.kicad_sch          (Power Supply)
- cm-conn1.kicad_sch     (CM4 Connector 1: power, USB, HDMI)
- cm-conn2.kicad_sch     (CM4 Connector 2: PCIe, Ethernet, GPIO, I2C)
- sata.kicad_sch         (ASM1061 PCIe-to-SATA)
- peripherals.kicad_sch  (RTC, LED, button)
Other:
- title: Granit — CM4/CM5 + Ethernet -> Granit — cm-conn2
Changed lines of the file:
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@@
 	(paper "A4")
 	(title_block
-		(title "Granit — CM4/CM5 + Ethernet")
+		(title "Granit — cm-conn2")
 		(date "2026-04-07")
 		(rev "0.1")
@@
 	(sheet_instances
 		(path "/"
-			(page "3")
+			(page "")
 		)
 	)

Commit message: CM4 connectors: add symbols/footprints, connect power pins
- Copy CM4 symbol and footprint from pedalboard-hw to granit library
- Remove all pedalboard library references
- Connect GND and +5V power pins on both connectors
- PSU GND ERC error resolved
- 0 ERC warnings, remaining errors are expected unconnected signal pins
Parts:
- added CM1: CM4, granit:Raspberry-Pi-4-Compute-Module, symbol granit:CM4
Connections:
- new net GND: CM1.107 (GND), CM1.108 (GND), CM1.113 (GND), CM1.114 (GND), CM1.119 (GND), CM1.120 (GND), CM1.125 (GND), CM1.126 (GND), CM1.131 (GND), CM1.132 (GND), CM1.137 (GND), CM1.138 (GND), CM1.144 (GND), CM1.150 (GND), CM1.155 (GND), CM1.156 (GND), CM1.161 (GND), CM1.162 (GND), CM1.167 (GND), CM1.168 (GND), CM1.173 (GND), CM1.174 (GND), CM1.179 (GND), CM1.180 (GND), CM1.185 (GND), CM1.186 (GND), CM1.191 (GND), CM1.192 (GND), CM1.197 (GND), CM1.198 (GND)

Commit message: CI: use KiBot dev branch with KiCad 10 support
KiBot 1.8.6 (dev) can parse KiCad 10 files.
Install from git dev branch + KiCad 10 PPA on ubuntu-latest.
Parts:
- CM1: footprint granit:Raspberry-Pi-4-Compute-Module -> Pedalboard Library:Raspberry-Pi-4-Compute-Module; symbol granit:CM4 -> pedalboard:CM4
Changed lines of the file:
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@@
 	)
 	(symbol
-		(lib_id "granit:CM4")
+		(lib_id "pedalboard:CM4")
 		(at -50.8 104.14 0)
 		(unit 2)
@@
 			)
 		)
-		(property "Footprint" "granit:Raspberry-Pi-4-Compute-Module"
+		(property "Footprint" "Pedalboard Library:Raspberry-Pi-4-Compute-Module"
 			(at 91.44 130.81 0)
 			(hide yes)
