File: hardware/cm-conn2.kicad_sch (KiCad schematic)
At the start: 1 part

Commit message: ERC: 0 errors, 0 warnings — fully clean
- Fix ASM1061 footprint reference (granit:QFN50P700X700X90-49N-D)
- Fix CM4 embedded symbol references (pedalboard → granit)
- Sync ASM1061 embedded symbol with library
- Remove dangling no-connect flags
- Re-add NC for barrel jack switch pin (J7 pin 3)
Parts:
- CM1: footprint Pedalboard Library:Raspberry-Pi-4-Compute-Module -> granit:Raspberry-Pi-4-Compute-Module; symbol pedalboard:CM4 -> granit:CM4
Changed lines of the file:
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@@
 	)
 	(symbol
-		(lib_id "pedalboard:CM4")
+		(lib_id "granit:CM4")
 		(at -50.8 104.14 0)
 		(unit 2)
@@
 			)
 		)
-		(property "Footprint" "Pedalboard Library:Raspberry-Pi-4-Compute-Module"
+		(property "Footprint" "granit:Raspberry-Pi-4-Compute-Module"
 			(at 91.44 130.81 0)
 			(hide yes)
